File: kicad_demo.sch (KiCad schematic (older format))
At the start: 35 parts, among them P1 pwr, P2 key, Q1 BC546, Q2 BC546, Q3 BC546, Y1 7030 kHz

Commit message: Upgrade to KiCAD 5.0.0
Parts:
- AE1: symbol Antenna -> kicad_demo-rescue:Antenna
- C1, C10, C11, C12, C13, C14, C2, C3, C4, C5, C6, C7, C8, C9: symbol C -> kicad_demo-rescue:C
- L1: symbol L_Core_Ferrite -> kicad_demo-rescue:L_Core_Ferrite
- L2, L3: symbol L -> kicad_demo-rescue:L
- P1, P2: symbol CONN_01X02 -> kicad_demo-rescue:CONN_01X02
- Q1, Q2, Q3: symbol Q_NPN_CBE -> kicad_demo-rescue:Q_NPN_CBE
- R1: symbol R -> kicad_demo-rescue:R
- W1, W10, W2, W3, W4, W5, W6, W7, W8, W9: symbol TEST_1P -> kicad_demo-rescue:TEST_1P
- Y1: symbol Crystal -> kicad_demo-rescue:Crystal
Connections:
- wire segments 56 -> 97
